File: Pololu_DRV8825/kicad/Pololu_DRV8825.kicad_pcb (KiCad board)
At the start: 2 copper layers, 100 x 60 mm, 23 parts, among them J1 CONN_01X02, J2 CONN_01X02, P1 CONN_01X10, P2 CONN_01X10, P3 CONN_02X10, P4 CONN_02X10, P5 CONN_01X04, P6 CONN_01X04, U1 MSP430G2553IN20, U2 LM2931Z-3.3/5.0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

Commit message: DRV8825 first routed board with mounting holes
Parts:
- added J3: CONN_01X02, Pin_Headers:Pin_Header_Straight_1x02, F.Cu at (124.1, 116.2)
- added REF**: 1pin, Connect:1pin, F.Cu at (160.0, 67.3)
- added REF**: 1pin, Connect:1pin, F.Cu at (69.3, 67.3)
- added REF**: 1pin, Connect:1pin, F.Cu at (69.3, 118.6)
- added REF**: 1pin, Connect:1pin, F.Cu at (147.1, 118.4)
- moved J2 5.98 mm to (77.0, 94.0)
- moved C1 4.26 mm to (110.7, 112.3)
- moved U2 3.24 mm to (107.2, 106.4)
- moved BT1 2.54 mm to (113.5, 117.0)
Connections:
- D1 pad 1: GND -> Net-(D1-Pad1)
- D2 pad 1: GND -> Net-(D1-Pad1)
- P3 pad 1: GND -> Net-(D1-Pad1)
- P3 pad 11: GND -> Net-(P3-Pad11)
- P3 pad 13: GND -> Net-(D1-Pad1)
- P3 pad 15: GND -> Net-(D1-Pad1)
- P3 pad 17: GND -> Net-(D1-Pad1)
- P3 pad 19: GND -> Net-(D1-Pad1)
- P3 pad 3: GND -> Net-(D1-Pad1)
- P3 pad 5: GND -> Net-(D1-Pad1)
- P3 pad 7: GND -> Net-(D1-Pad1)
- P3 pad 9: GND -> Net-(D1-Pad1)
Routing:
- net GND: track 0.00 -> 198.5 mm
- net +3V3: track 0.00 -> 166.2 mm
- net /STEP2: track 0.00 -> 86.7 mm
- net +12V: track 0.00 -> 84.8 mm
- net Net-(J2-Pad2): track 0.00 -> 72.4 mm
- net /IN9: track 0.00 -> 64.3 mm
- net /STEP1: track 0.00 -> 63.4 mm
- net /IN2: track 0.00 -> 60.6 mm
- net /IN3: track 0.00 -> 60.5 mm
- net /IN5: track 0.00 -> 60.5 mm
- net /IN4: track 0.00 -> 60.5 mm
- net /IN8: track 0.00 -> 59.7 mm
- net /IN1: track 0.00 -> 59.3 mm
- net Net-(D1-Pad1): track 0.00 -> 56.5 mm
- net /IN7: track 0.00 -> 55.0 mm
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Other:
- net class Big Power added: clearance 0.3, trace_width 0.6, via_dia 0.9, via_drill 0.4
- net class Default: via_dia 0.6 -> 0.9
- net class Power: trace_width 0.8 -> 0.3; via_dia 0.6 -> 0.8
- rule via_min_size: 0.4 -> 0.8
- board text added: "+"
- board text added: "G"
